Commit message: Yolo_reco

File: src/arm_dm_description/urdf/arm_dm_description.urdf (robot description, URDF)
Before this commit: robot arm_dm_description, 7 links, 6 joints
Links:
- added link tcp_link; visual sphere radius=0.01
- link base_link: mass 0.70252 -> 0.976
- link link1: mass 0.12465 -> 0.138
- link link2: mass 0.83418 -> 1.379
- link link3: mass 0.49894 -> 0.727
- link link4: mass 0.17215 -> 0.370
- link link5: mass 0.38198 -> 0.391
- link link6: mass 0.0045985 -> 0.179
Joints:
- added joint tool_flange_to_tcp: type fixed, parent link6, child tcp_link, origin xyz=0.0 0.09 0.0 rpy=0 0 0
